Commit message: Define first functional master branch
  - Specify simulation parameters to achieve close to real time simulation
  - Enforce ROS conventions on Python executable naming, and module installation
  - Implement a simple waypoint following node

File: src/deedee_description/urdf/deedee.xacro (robot description, xacro)
@@ -82,5 +82,5 @@
               rpy="0 0 0"
       />
-      <limit effort="30" velocity="1.0"/>
+      <limit effort="2000" velocity="4.0"/>
     </joint>
     <gazebo reference="${prefix}_wheel">

Commit message: Fiddle with gazebo simulation parameters

File: src/deedee_description/urdf/deedee.xacro (robot description, xacro)
@@ -11,4 +11,7 @@
   </material>
   <!-- #################    MACROS     ##################### -->
+  <xacro:property name="baseweight" value="50.0" />
+  <xacro:property name="wheelweight" value="10.0" />
+  <xacro:property name="castorweight" value="5" />
   <xacro:property name="basewidth" value="0.4" />
   <xacro:property name="baselength" value="0.6" />
@@ -22,10 +25,10 @@
     <inertial>
       <mass value="${mass}" />
-      <inertia ixx="${((dy*dy)+(dz*dz))/3}"
+      <inertia ixx="${mass*((dy*dy)+(dz*dz))/3}"
                ixy="0.0"
                ixz="0.0"
-               iyy="${(dx*dx+dz*dz)/3}"
+               iyy="${mass*(dx*dx+dz*dz)/3}"
                iyz="0.0"
-               izz="${(dx*dx+dy*dy)/3}"
+               izz="${mass*(dx*dx+dy*dy)/3}"
       />
     </inertial>
@@ -34,10 +37,10 @@
     <inertial>
       <mass value="${mass}" />
-      <inertia ixx="${radius*radius/2}"
+      <inertia ixx="${mass*radius*radius/2}"
                ixy="0.0"
                ixz="0.0"
-               iyy="${radius*radius/4 + height*height/3}"
+               iyy="${mass*radius*radius/4 + height*height/3}"
                iyz="0.0"
-               izz="${radius*radius/4 + height*height/3}" />
+               izz="${mass*radius*radius/4 + height*height/3}" />
     </inertial>
   </xacro:macro>
@@ -45,10 +48,10 @@
     <inertial>
       <mass value="${mass}" />
-      <inertia ixx="${2*radius*radius/3}"
+      <inertia ixx="${mass*2*radius*radius/3}"
                ixy="0.0"
                ixz="0.0"
-               iyy="${2*radius*radius/3}"
+               iyy="${mass*2*radius*radius/3}"
                iyz="0.0"
-               izz="${2*radius*radius/3}" />
+               izz="${mass*2*radius*radius/3}" />
     </inertial>
   </xacro:macro>
@@ -64,12 +67,12 @@
       </visual>
       <collision>
-        <origin xyz="0 0 0" rpy="${side*pi/2} 0 0" />
+        <origin xyz="0 0 0" rpy="${pi/2} 0 0" />
         <geometry>
           <cylinder radius="${wheelradius}" length="${wheelwidth}"/>
         </geometry>
       </collision>
-      <xacro:cylinder_inertial mass="0.2"
-                            radius="${wheelradius}"
-                            height="${wheelwidth}"/>
+      <cylinder_inertial mass="${wheelweight}"
+                         radius="${wheelradius}"
+                         height="${wheelwidth}"/>
     </link>
     <joint name="${prefix}_wheel_joint" type="continuous">
@@ -83,10 +86,12 @@
       />
       <limit effort="2000" velocity="4.0"/>
+      <dynamics damping="0.7"/>
     </joint>
     <gazebo reference="${prefix}_wheel">
+      <dampignFactor value="0.5"/>
       <mu1 value="200.0"/>
-      <mu2 value="100.0"/>
-      <kp value="10000000.0" />
-      <kd value="1.0" />
+      <mu2 value="200.0"/>
+      <kp value="100000.0"/>
+      <kp value="1.0"/>
       <material>Gazebo/Grey</material>
     </gazebo>
@@ -115,8 +120,8 @@
       </geometry>
     </collision>
-    <xacro:box_inertial mass="1"
-                        dx="${baselength}"
-                        dy="${basewidth}"
-                        dz="${baseheight}"
+    <box_inertial mass="${baseweight}"
+                  dx="${baselength}"
+                  dy="${basewidth}"
+                  dz="${baseheight}"
     />
   </link>
@@ -136,6 +141,6 @@
       </geometry>
     </collision>
-    <xacro:sphere_inertial mass="1"
-                           radius="${castorradius}"
+    <sphere_inertial mass="${castorweight}"
+                     radius="${castorradius}"
     />
   </link>
@@ -151,6 +156,6 @@
   </gazebo>
   <!-- Wheels -->
-  <xacro:wheel prefix="left" side="1"/>
-  <xacro:wheel prefix="right" side="-1"/>
+  <wheel prefix="left" side="1"/>
+  <wheel prefix="right" side="-1"/>
   <!-- ###############     Gazebo link     ############### -->
   <gazebo>

Commit message: Modify physics settings of joints

File: src/deedee_description/urdf/deedee.xacro (robot description, xacro)
@@ -76,4 +76,8 @@
                          height="${wheelwidth}"/>
     </link>
+    <gazebo reference="${prefix}_wheel">
+      <dampingFactor>0.5</dampingFactor>
+      <material>Gazebo/Grey</material>
+    </gazebo>
     <joint name="${prefix}_wheel_joint" type="continuous">
       <axis xyz="0 1 0" rpy="0 0 0" />
@@ -86,12 +90,8 @@
       />
       <limit effort="2000" velocity="4.0"/>
-      <dynamics damping="0.7"/>
+      <dynamics damping="0.7" friction="1.0"/>>
     </joint>
-    <gazebo reference="${prefix}_wheel">
-      <dampignFactor value="0.5"/>
-      <mu1 value="200.0"/>
-      <mu2 value="200.0"/>
-      <kp value="100000.0"/>
-      <kp value="1.0"/>
+    <gazebo reference="${prefix}_wheel_joint">
+      <dampingFactor>0.5</dampingFactor>
       <material>Gazebo/Grey</material>
     </gazebo>

Commit message: Fiddle with simulation settings and add willowgarage

File: src/deedee_description/urdf/deedee.xacro (robot description, xacro)
@@ -11,7 +11,7 @@
   </material>
   <!-- #################    MACROS     ##################### -->
-  <xacro:property name="baseweight" value="50.0" />
-  <xacro:property name="wheelweight" value="10.0" />
-  <xacro:property name="castorweight" value="5" />
+  <xacro:property name="baseweight" value="2.0" />
+  <xacro:property name="wheelweight" value="0.5" />
+  <xacro:property name="castorweight" value="0.4" />
   <xacro:property name="basewidth" value="0.4" />
   <xacro:property name="baselength" value="0.6" />
@@ -77,5 +77,8 @@
     </link>
     <gazebo reference="${prefix}_wheel">
-      <dampingFactor>0.5</dampingFactor>
+      <mu1 value="200.0"/>
+      <mu2 value="100.0"/>
+      <kp value="10000000.0" />
+      <kd value="1.0" />
       <material>Gazebo/Grey</material>
     </gazebo>
@@ -90,8 +93,8 @@
       />
       <limit effort="2000" velocity="4.0"/>
-      <dynamics damping="0.7" friction="1.0"/>>
+      <dynamics damping="0.3" friction="30.0"/>>
     </joint>
     <gazebo reference="${prefix}_wheel_joint">
-      <dampingFactor>0.5</dampingFactor>
+      <dampingFactor>0.1</dampingFactor>
       <material>Gazebo/Grey</material>
     </gazebo>
